File: 01-hardware/walkeeg_v3.0/walkeeg_v3.0.kicad_sch (KiCad schematic)
At the start: 0 parts

Commit message: update SCH design
Other:
- added sheet MotherBroad (walkeeg_v3.0_mother_broad.kicad_sch)
- added sheet Peripherals (walkeeg_v3.0_peripherals.kicad_sch)
- note added: "Peripherals = 电源/USB/存储 (AMS1117, USB 磁珠防护, SPI Flash, SD, CH340)"
- note added: "WalkEEG v3.0 —— 8 通道便携脑电采集板"
- note added: "主控: nRF52840 模块 (青风) | 模拟前端: 8x AD8232 + ADS1293"
- note added: "外设: SPI Flash (W25Q80) / MicroSD / CH340C USB 串口"
- note added: "页面说明: MotherBroad = 主控接口/模拟前端 (J1 J2 排针, 8x AD8232, ADS1293, 测试点)"
Changed lines of the file:
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@@
 	(generator_version "10.0")
 	(paper "A4")
+	(text "           Peripherals = 电源/USB/存储 (AMS1117, USB 磁珠防护, SPI Flash, SD, CH340)"
+		(exclude_from_sim no)
+		(at 85.598 67.582 0)
+		(effects
+			(font
+				(size 2 2)
+			)
+			(justify left)
+		)
+	)
+	(text "WalkEEG v3.0  ——  8 通道便携脑电采集板"
+		(exclude_from_sim no)
+		(at 87.63 56.896 0)
+		(effects
+			(font
+				(size 3.5 3.5)
+			)
+			(justify left)
+		)
+	)
+	(text "主控: nRF52840 模块 (青风)  |  模拟前端: 8x AD8232 + ADS1293"
+		(exclude_from_sim no)
+		(at 85.598 84.582 0)
+		(effects
+			(font
+				(size 2 2)
+			)
+			(justify left)
+		)
+	)
+	(text "页面说明:  MotherBroad = 主控接口/模拟前端 (J1 J2 排针, 8x AD8232, ADS1293, 测试点)"
+		(exclude_from_sim no)
+		(at 85.598 72.582 0)
+		(effects
+			(font
+				(size 2 2)
+			)
+			(justify left)
+		)
+	)
+	(text "外设: SPI Flash (W25Q80) / MicroSD / CH340C USB 串口"
+		(exclude_from_sim no)
+		(at 85.598 79.582 0)
+		(effects
+			(font
+				(size 2 2)
+			)
+			(justify left)
+		)
+	)
+	(sheet
+		(at 92.38 94.6)
+		(size 45.72 30.48)
+		(exclude_from_sim no)
+		(in_bom yes)
+		(on_board yes)
+		(dnp no)
+		(stroke
+			(width 0.1524)
+			(type solid)
+		)
+		(fill
+			(color 255 255 255 0)
+		)
+		(property "Sheetname" "MotherBroad"
+			(at 13.97 -2.032 0)
+			(show_name no)
+			(do_not_autoplace no)
+			(effects
+				(font
+					(size 1.27 1.27)
+				)
+				(justify left bottom)
+			)
+		)
+		(property "Sheetfile" "walkeeg_v3.0_mother_broad.kicad_sch"
+			(at 15.24 -27.94 0)
+			(show_name no)
+			(do_not_autoplace no)
+			(effects
+				(font
+					(size 1.27 1.27)
+				)
+				(justify left top)
+			)
+		)
+		(instances
+			(project "walkeeg_v3.0"
+				(path "/e697d0ae-258a-4ffe-a80f-5c30fd5207ba"
+					(page "2")
+				)
+			)
+		)
+	)
+	(sheet
+		(at 161.27 94.6)
+		(size 45.72 30.48)
+		(exclude_from_sim no)
+		(in_bom yes)
+		(on_board yes)
+		(dnp no)
+		(stroke
+			(width 0.1524)
+			(type solid)
+		)
+		(fill
+			(color 255 255 255 0)
+		)
+		(property "Sheetname" "Peripherals"
+			(at 22.86 -2.032 0)
+			(show_name no)
+			(do_not_autoplace no)
+			(effects
+				(font
+					(size 1.27 1.27)
+				)
+				(justify left bottom)
+			)
+		)
+		(property "Sheetfile" "walkeeg_v3.0_peripherals.kicad_sch"
+			(at 24.13 -27.94 0)
+			(show_name no)
+			(do_not_autoplace no)
+			(effects
+				(font
+					(size 1.27 1.27)
+				)
+				(justify left top)
+			)
+		)
+		(instances
+			(project "walkeeg_v3.0"
+				(path "/e697d0ae-258a-4ffe-a80f-5c30fd5207ba"
+					(page "3")
+				)
+			)
+		)
+	)
 	(sheet_instances
 		(path "/"
