File: 01-hardware/walkeeg_v3.0/walkeeg_v3.0_mother_broad.kicad_sch (KiCad schematic)
At the start: 72 parts, among them J1 Con_2_core, J10 AD8232_connector, J11 ADS1293, J15 Conn_02x05_Odd_Even, J2 Con_2_core, J3 AD8232_connector, J4 AD8232_connector, J5 AD8232_connector, J6 AD8232_connector, J7 AD8232_connector, J8 AD8232_connector, J9 AD8232_connector, SW1 SW_Push

Commit message: finish DRC
Parts:
- renumbered R_SDN to R11, R_LO+ to R12, R_LO- to R13
Connections:
- no-connect marks 0 -> 2
Changed lines of the file:
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@@
 		)
 	)
-	(global_label "P0.19{slash}LED2"
-		(shape passive)
+	(label "P0.19{slash}LED2"
 		(at 49.53 185.42 0)
 		(effects
@@
 			(justify left)
 		)
-		(property "Intersheetrefs" "${INTERSHEET_REFS}"
-			(at 49.53 185.42 0)
-			(hide yes)
-			(show_name no)
-			(do_not_autoplace no)
-			(effects
-				(font
-					(size 1.27 1.27)
-				)
-			)
-		)
 	)
 	(global_label "GND"
@@
 		)
 	)
-	(global_label "P1.01"
-		(shape passive)
+	(label "P1.01"
 		(at 76.2 160.02 180)
 		(effects
@@
 			(justify right)
 		)
-		(property "Intersheetrefs" "${INTERSHEET_REFS}"
-			(at 76.2 160.02 0)
-			(hide yes)
-			(show_name no)
-			(do_not_autoplace no)
-			(effects
-				(font
-					(size 1.27 1.27)
-				)
-				(justify left)
-			)
-		)
 	)
-	(global_label "P0.17{slash}LED1"
-		(shape passive)
+	(label "P0.17{slash}LED1"
 		(at 30.48 185.42 0)
 		(effects
@@
 			(justify left)
 		)
-		(property "Intersheetrefs" "${INTERSHEET_REFS}"
-			(at 30.48 185.42 0)
-			(hide yes)
-			(show_name no)
-			(do_not_autoplace no)
-			(effects
-				(font
-					(size 1.27 1.27)
-				)
-			)
-		)
 	)
 	(global_label "P0.26"
@@
 		(dnp no)
 		(fields_autoplaced yes)
-		(property "Reference" "R_LO-"
-			(at 240.03 146.05 0)
+		(property "Reference" "R13"
+			(at 247.65 142.2399 0)
 			(show_name no)
 			(do_not_autoplace no)
@@
 					(size 1.27 1.27)
 				)
+				(justify left)
 			)
 		)
 		(property "Value" "10k"
-			(at 250.19 140.97 0)
+			(at 247.65 144.7799 0)
 			(show_name no)
 			(do_not_autoplace no)
@@
 					(size 1.27 1.27)
 				)
+				(justify left)
 			)
 		)
@@
 			(project "walkeeg_v3.0"
 				(path "/e697d0ae-258a-4ffe-a80f-5c30fd5207ba/76b461a0-7f1d-4d4a-9fb9-de3608d0b7fc"
-					(reference "R_LO-")
+					(reference "R13")
 					(unit 1)
 				)
@@
 		(dnp no)
 		(fields_autoplaced yes)
-		(property "Reference" "R_SDN"
-			(at 240.03 90.17 0)
+		(property "Reference" "R11"
+			(at 247.65 86.3599 0)
 			(show_name no)
 			(do_not_autoplace no)
@@
 					(size 1.27 1.27)
 				)
+				(justify left)
 			)
 		)
 		(property "Value" "10k"
-			(at 250.19 85.09 0)
+			(at 247.65 88.8999 0)
 			(show_name no)
 			(do_not_autoplace no)
@@
 					(size 1.27 1.27)
 				)
+				(justify left)
 			)
 		)
@@
 			(project "walkeeg_v3.0"
 				(path "/e697d0ae-258a-4ffe-a80f-5c30fd5207ba/76b461a0-7f1d-4d4a-9fb9-de3608d0b7fc"
-					(reference "R_SDN")
+					(reference "R11")
 					(unit 1)
 				)
@@
 		(dnp no)
 		(fields_autoplaced yes)
-		(property "Reference" "R_LO+"
-			(at 240.03 119.38 0)
+		(property "Reference" "R12"
+			(at 247.65 115.5699 0)
 			(show_name no)
 			(do_not_autoplace no)
@@
 					(size 1.27 1.27)
 				)
+				(justify left)
 			)
 		)
 		(property "Value" "10k"
-			(at 250.19 114.3 0)
+			(at 247.65 118.1099 0)
 			(show_name no)
 			(do_not_autoplace no)
@@
 					(size 1.27 1.27)
 				)
+				(justify left)
 			)
 		)
@@
 			(project "walkeeg_v3.0"
 				(path "/e697d0ae-258a-4ffe-a80f-5c30fd5207ba/76b461a0-7f1d-4d4a-9fb9-de3608d0b7fc"
-					(reference "R_LO+")
+					(reference "R12")
 					(unit 1)
 				)
@@
 		)
 	)
+	(no_connect
+		(at 243.84 62.23 0)
+	)
+	(no_connect
+		(at 256.54 62.23 0)
+	)
 )
