File: 01-hardware/walkeeg_v3.0/walkeeg_v3.0_peripherals.kicad_sch (KiCad schematic)
At the start: 31 parts, among them J12 USB_B_Micro_UART, J13 USB_B_Micro, U5 W25Q80DVSSIG, U6 Micro_SD_Card, U7 CH340C, U8 AMS1117-3.3, U9 PRTR5V0U2X

Commit message: finish DRC
Connections:
- no-connect marks 0 -> 6
Changed lines of the file:
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@@
 		)
 	)
-	(label "VBUS"
-		(at 25.4 146.05 0)
-		(effects
-			(font
-				(size 1.27 1.27)
-			)
-			(justify left)
-		)
-	)
 	(label "CH340_D-"
 		(at 161.29 48.26 0)
@@
 		)
 	)
+	(no_connect
+		(at 193.04 88.9 0)
+	)
+	(no_connect
+		(at 213.36 96.52 0)
+	)
+	(no_connect
+		(at 213.36 99.06 0)
+	)
+	(no_connect
+		(at 213.36 101.6 0)
+	)
+	(no_connect
+		(at 213.36 104.14 0)
+	)
+	(no_connect
+		(at 157.48 50.8 0)
+	)
 )

Commit message: sch update to pcb
unfinished
Parts:
- U5: footprint W25Q80DVSSIG:SOIC8-FLASH -> Package_SO:SOIC-8_3.9x4.9mm_P1.27mm; symbol W25Q80DVSSIG:W25Q80DVSSIG -> w25q80:W25Q80DVSSIG
- U6: footprint (none) -> Connector_Card:microSD_HC_Hirose_DM3AT-SF-PEJM5
Changed lines of the file:
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@@
 	)
 	(symbol
-		(lib_id "W25Q80DVSSIG:W25Q80DVSSIG")
+		(lib_id "w25q80:W25Q80DVSSIG")
 		(at 82.55 55.88 0)
 		(unit 1)
@@
 			)
 		)
-		(property "Footprint" "W25Q80DVSSIG:SOIC8-FLASH"
+		(property "Footprint" "Package_SO:SOIC-8_3.9x4.9mm_P1.27mm"
 			(at 82.55 55.88 0)
 			(hide yes)
@@
 			)
 		)
-		(property "Footprint" ""
+		(property "Footprint" "Connector_Card:microSD_HC_Hirose_DM3AT-SF-PEJM5"
 			(at 91.44 107.95 0)
 			(hide yes)
@@
 	)
 	(no_connect
-		(at 193.04 88.9 0)
+		(at 193.04 88.9)
 	)
 	(no_connect
-		(at 213.36 96.52 0)
+		(at 213.36 96.52)
 	)
 	(no_connect
-		(at 213.36 99.06 0)
+		(at 213.36 99.06)
 	)
 	(no_connect
-		(at 213.36 101.6 0)
+		(at 213.36 101.6)
 	)
 	(no_connect
-		(at 213.36 104.14 0)
+		(at 213.36 104.14)
 	)
 	(no_connect
-		(at 157.48 50.8 0)
+		(at 157.48 50.8)
 	)
 )
