File: 01-hardware/walkeeg_v3.0/walkeeg_v3.0.kicad_pcb (KiCad board)
At the start: 2 copper layers, 103 parts, among them J1 Con_2_core, J10 AD8232_connector, J11 ADS1293, J12 USB_B_Micro_UART, J13 USB_B_Micro, J15 Conn_02x05_Odd_Even, J2 Con_2_core, J3 AD8232_connector, J4 AD8232_connector, J5 AD8232_connector, J6 AD8232_connector, J7 AD8232_connector, J8 AD8232_connector, J9 AD8232_connector, SW1 SW_Push, U5 W25Q80DVSSIG, U6 Micro_SD_Card, U7 CH340C, U8 AMS1117-3.3, U9 PRTR5V0U2X

Commit message: commit pcb design(not finish)
Parts:
- added H1: H1, MountingHole_3.2mm_M3, F.Cu at (68.0, 52.0)
- added H2: H2, MountingHole_3.2mm_M3, F.Cu at (163.0, 52.0)
- added H3: H3, MountingHole_3.2mm_M3, F.Cu at (163.0, 177.0)
- moved TP27 132.5 mm to (149.0, 87.5)
- moved TP36 123.8 mm to (153.0, 100.2)
- moved TP34 119.7 mm to (153.0, 97.7)
- moved TP35 119.4 mm to (149.0, 97.7)
- moved R12 116.9 mm to (152.7, 139.0), turned to 180 degrees
- moved TP32 116.0 mm to (153.0, 95.1)
- moved TP33 115.3 mm to (149.0, 95.1)
- moved TP30 112.5 mm to (153.0, 92.6)
- moved TP31 111.5 mm to (149.0, 92.6)
- moved TP44 111.3 mm to (153.0, 110.4)
- moved TP45 110.7 mm to (149.0, 110.4)
- moved R10 110.3 mm to (107.8, 177.7), turned to 180 degrees
- moved TP28 109.2 mm to (153.0, 90.0)
- moved TP29 108.0 mm to (149.0, 90.0)
- moved TP42 107.8 mm to (153.0, 107.8)
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Routing:
- net +3V3: track 0.00 -> 489.4 mm, vias 0 -> 4
- net /MotherBroad/P0.24/SDN: track 0.00 -> 319.8 mm, vias 0 -> 7
- net /MotherBroad/P1.00/ALARMB: track 0.00 -> 176.4 mm, vias 0 -> 8
- net /MotherBroad/P1.07/RSTB: track 0.00 -> 155.2 mm, vias 0 -> 1
- net /MotherBroad/P1.05/CSB: track 0.00 -> 154.8 mm, vias 0 -> 5
- net /MotherBroad/P1.04/SDO: track 0.00 -> 150.0 mm, vias 0 -> 4
- net /MotherBroad/P1.03/SCLK: track 0.00 -> 147.2 mm, vias 0 -> 5
- net /MotherBroad/P1.06/DRDYB: track 0.00 -> 141.8 mm, vias 0 -> 2
- net P0.06/TXD: track 0.00 -> 133.2 mm, vias 0 -> 6
- net D+: track 0.00 -> 132.6 mm, vias 0 -> 1
- net /MotherBroad/P0.31/AIN7: track 0.00 -> 132.4 mm, vias 0 -> 1
- net /MotherBroad/P0.30/AIN6: track 0.00 -> 123.6 mm, vias 0 -> 3
- net /MotherBroad/P0.28/AIN4: track 0.00 -> 119.8 mm, vias 0 -> 1
- net /MotherBroad/P0.26/SCL: track 0.00 -> 117.0 mm, vias 0 -> 3
- net /MotherBroad/P0.05/AIN3: track 0.00 -> 64.2 mm, vias 0 -> 2
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Other:
- board outline added: 107 x 137 mm
- board text added: "2026-08-24"
- board text added: "8-CH EEG nRF52840"
- board text added: "WalkEEG v3.0"
